File: Angle-from-as5600/Angle-from-as5600.kicad_sch (KiCad schematic)
At the start: 10 parts, among them J1 Conn_01x03_Pin, J3 Conn_01x05_Socket, U1 AS5600

Commit message: fix kicad files
fix pin pitch
Parts:
- J3: footprint Connector_PinHeader_1.00mm:PinHeader_1x05_P1.00mm_Horizontal -> Connector_PinHeader_2.54mm:PinHeader_1x05_P2.54mm_Horizontal
- U2: footprint Package_SO:SSOP-20_4.4x6.5mm_P0.65mm -> Package_SO:SSOP-20_4.4x6.5mm_P0.65mm_bigpad
